File: PCB/Detectors.brd (EAGLE design)
At the start: 38.1 x 44.1 mm, 12 parts, among them IC1 LM4041A12DBZ, J1 RJ11-4X

Commit message: updated PCB and scematic
Parts:
- moved R4 28.9 mm to (26.7, 3.56), turned to 90 degrees
- moved R1 11.7 mm to (39.4, 11.4)
- moved R3 11.7 mm to (39.4, 19.1)
- moved IC1 9.16 mm to (11.4, 3.81), turned to 90 degrees
- moved R2 8.89 mm to (39.4, 3.81)
- moved B1 6.35 mm to (17.8, 25.4)
- moved R5 5.99 mm to (21.2, 3.05)
- moved LED1 3.81 mm to (33.0, 3.81), turned to 180 degrees
- moved LED2 3.81 mm to (33.0, 19.1), turned to 180 degrees
- moved LED3 3.81 mm to (33.0, 11.4), turned to 180 degrees
- moved R6 3.70 mm to (15.4, 4.06), turned to 270 degrees
Connections:
- net N$1: now also J1.3
- net N$8: no longer J1.5
- net N$9: now also J1.4; no longer J1.6
Routing:
- net N$9: track 15.0 -> 58.2 mm
- net N$1: track 11.3 -> 53.0 mm
- net N$8: track 55.7 -> 21.4 mm
- net N$5: track 0.00 -> 15.4 mm
- net N$6: track 0.00 -> 10.3 mm
- net N$7: track 0.00 -> 7.42 mm
- net N$4: track 0.00 -> 4.13 mm
- net N$3: track 0.00 -> 4.13 mm
- net N$2: track 0.00 -> 4.13 mm
Other:
- board size 38.1 x 44.1 mm -> 38.1 x 47.9 mm
- board text added: "This detector was, Built by Robo SciOly, This is a haiku"
